Commit message: Update robot_final.xacro

File: urdf/robot_final.xacro (robot description, xacro)
@@ -128,4 +128,78 @@
     <child link="caster2_link" />
     <axis xyz="0.0028853 -0.031751 -0.99949" />
+  </joint>
+  ----------------------------------------------
+ <joint name="camera_joint" type="fixed">
+    <axis xyz="0 1 0" />
+    <origin
+        xyz="0.16 0 0.20"
+        rpy="2.0 0 1.57" />
+    <parent
+      link="base_link" />
+    <child
+      link="camera_link" />
+  </joint>
+<link name="camera_link">
+    <visual>
+      <origin
+        xyz="0 0 0"
+        rpy="0 0 0" />
+      <geometry>
+        <mesh
+          filename="package://robot_final/meshes/asus_xtion_pro_live_camera.dae" scale="0.001 0.001 0.001"/>
+      </geometry>
+    </visual>
+    <collision>
+      <origin
+        xyz="0 0 0"
+        rpy="0 0 0" />
+      <geometry>
+        <mesh
+          filename="package://robot_final/meshes/asus_xtion_pro_live_camera.dae" scale="0.001 0.001 0.001" />
+      </geometry>
+    </collision>
+  </link>
+<joint name="camera_point_joint" type="fixed">
+    <axis xyz="0 1 0" />
+    <origin
+        xyz="0.023 0 0.015"
+        rpy="0 0 0" />
+    <parent
+      link="camera_link" />
+    <child
+      link="camera_point_link" />
+  </joint>
+<link name="camera_point_link">
+    <visual>
+      <origin
+        xyz="0 0 0"
+        rpy="0 0 0" />
+    </visual>
+  </link>
+  <link name="hokuyo_link">
+    <collision>
+      <origin xyz="0 0 0" rpy="0 0 0"/>
+      <geometry>
+    <box size="0.1 0.1 0.1"/>
+      </geometry>
+    </collision>
+    <visual>
+      <origin xyz="0 0 0" rpy="0 0 0"/>
+      <geometry>
+        <mesh filename="package://simple_robot_LIDAR/meshes/hokuyo.dae"/>
+      </geometry>
+    </visual>
+    <inertial>
+      <mass value="1e-5" />
+      <origin xyz="0 0 0" rpy="0 0 0"/>
+      <inertia ixx="1e-6" ixy="0" ixz="0" iyy="1e-6" iyz="0" izz="1e-6" />
+    </inertial>
+  </link>
+  <joint name="hokuyo_joint" type="fixed">
+    <axis xyz="0 1 0" />
+    <origin xyz="0 0 0.25" rpy="0 0 0"/>
+    <parent link="base_link"/>
+    <child link="hokuyo_link"/>
+	 <dynamics damping="0.7"/>
   </joint>
   <transmission name="left_wheel_transmission">

Commit message: Add files via upload

File: urdf/robot_final.xacro (robot description, xacro)
@@ -25,24 +25,4 @@
     </collision>
   </link>
-  <link name="left_wheel_link">
-    <inertial>
-      <origin xyz="0 0 0"/>
-      <mass value="0.01" />
-      <inertia ixx="0.001" ixy="0.0" ixz="0.0"
-        iyy="0.001" iyz="0.0" izz="0.001" />
-    </inertial>
-    <visual>
-      <origin xyz="0 0 0" rpy="0 0 0" />
-      <geometry>
-        <mesh filename="package://robot_final/meshes/left_wheel_link.STL" />
-      </geometry>
-    </visual>
-    <collision>
-      <origin xyz="0 0 0" rpy="0 0 0" />
-      <geometry>
-        <mesh filename="package://robot_final/meshes/left_wheel_link.STL" />
-      </geometry>
-    </collision>
-  </link>
   <joint name="left_wheel_joint" type="continuous">
     <origin xyz="0 -0.1005 0.09" rpy="1.5708 0 0" />
@@ -51,5 +31,5 @@
     <axis xyz="0 0 1" />
   </joint>
-  <link name="right_wheel_link">
+  <link name="left_wheel_link">
     <inertial>
       <origin xyz="0 0 0"/>
@@ -61,11 +41,11 @@
       <origin xyz="0 0 0" rpy="0 0 0" />
       <geometry>
-        <mesh filename="package://robot_final/meshes/right_wheel_link.STL" />
-      </geometry>
-    </visual>
-    <collision>
-      <origin xyz="0 0 0" rpy="0 0 0" />
-      <geometry>
-        <mesh filename="package://robot_final/meshes/right_wheel_link.STL" />
+        <mesh filename="package://robot_final/meshes/left_wheel_link.STL" />
+      </geometry>
+    </visual>
+    <collision>
+      <origin xyz="0 0 0" rpy="0 0 0" />
+      <geometry>
+        <mesh filename="package://robot_final/meshes/left_wheel_link.STL" />
       </geometry>
     </collision>
@@ -77,21 +57,21 @@
     <axis xyz="0 0 1" />
   </joint>
-  <link name="caster1_link">
-    <inertial>
-      <origin xyz="0 0 0" />
-      <mass value="0.01" />
-      <inertia ixx="0.001" ixy="0.0" ixz="0.0"
-        iyy="0.001" iyz="0.0" izz="0.001" />
-    </inertial>
-    <visual>
-      <origin xyz="0 0 0" rpy="0 0 0" />
-      <geometry>
-        <mesh filename="package://robot_final/meshes/caster1_link.STL" />
-      </geometry>
-    </visual>
-    <collision>
-      <origin xyz="0 0 0" rpy="0 0 0" />
-      <geometry>
-        <mesh filename="package://robot_final/meshes/caster1_link.STL" />
+  <link name="right_wheel_link">
+    <inertial>
+      <origin xyz="0 0 0"/>
+      <mass value="0.01" />
+      <inertia ixx="0.001" ixy="0.0" ixz="0.0"
+        iyy="0.001" iyz="0.0" izz="0.001" />
+    </inertial>
+    <visual>
+      <origin xyz="0 0 0" rpy="0 0 0" />
+      <geometry>
+        <mesh filename="package://robot_final/meshes/right_wheel_link.STL" />
+      </geometry>
+    </visual>
+    <collision>
+      <origin xyz="0 0 0" rpy="0 0 0" />
+      <geometry>
+        <mesh filename="package://robot_final/meshes/right_wheel_link.STL" />
       </geometry>
     </collision>
@@ -103,5 +83,5 @@
     <axis xyz="0 0 1" />
   </joint>
-  <link name="caster2_link">
+  <link name="caster1_link">
     <inertial>
       <origin xyz="0 0 0" />
@@ -113,11 +93,11 @@
       <origin xyz="0 0 0" rpy="0 0 0" />
       <geometry>
-        <mesh filename="package://robot_final/meshes/caster2_link.STL" />
-      </geometry>
-    </visual>
-    <collision>
-      <origin xyz="0 0 0" rpy="0 0 0" />
-      <geometry>
-        <mesh filename="package://robot_final/meshes/caster2_link.STL" />
+        <mesh filename="package://robot_final/meshes/caster1_link.STL" />
+      </geometry>
+    </visual>
+    <collision>
+      <origin xyz="0 0 0" rpy="0 0 0" />
+      <geometry>
+        <mesh filename="package://robot_final/meshes/caster1_link.STL" />
       </geometry>
     </collision>
@@ -129,6 +109,25 @@
     <axis xyz="0.0028853 -0.031751 -0.99949" />
   </joint>
-  ----------------------------------------------
- <joint name="camera_joint" type="fixed">
+  <link name="caster2_link">
+    <inertial>
+      <origin xyz="0 0 0" />
+      <mass value="0.01" />
+      <inertia ixx="0.001" ixy="0.0" ixz="0.0"
+        iyy="0.001" iyz="0.0" izz="0.001" />
+    </inertial>
+    <visual>
+      <origin xyz="0 0 0" rpy="0 0 0" />
+      <geometry>
+        <mesh filename="package://robot_final/meshes/caster2_link.STL" />
+      </geometry>
+    </visual>
+    <collision>
+      <origin xyz="0 0 0" rpy="0 0 0" />
+      <geometry>
+        <mesh filename="package://robot_final/meshes/caster2_link.STL" />
+      </geometry>
+    </collision>
+  </link>
+  <joint name="camera_joint" type="fixed">
     <axis xyz="0 1 0" />
     <origin
@@ -140,5 +139,5 @@
       link="camera_link" />
   </joint>
-<link name="camera_link">
+  <link name="camera_link">
     <visual>
       <origin
@@ -160,39 +159,11 @@
     </collision>
   </link>
-<joint name="camera_point_joint" type="fixed">
+  <joint name="camera_point_joint" type="fixed">
     <axis xyz="0 1 0" />
-    <origin
-        xyz="0.023 0 0.015"
-        rpy="0 0 0" />
-    <parent
-      link="camera_link" />
-    <child
-      link="camera_point_link" />
-  </joint>
-<link name="camera_point_link">
-    <visual>
-      <origin
-        xyz="0 0 0"
-        rpy="0 0 0" />
-    </visual>
-  </link>
-  <link name="hokuyo_link">
-    <collision>
-      <origin xyz="0 0 0" rpy="0 0 0"/>
-      <geometry>
-    <box size="0.1 0.1 0.1"/>
-      </geometry>
-    </collision>
-    <visual>
-      <origin xyz="0 0 0" rpy="0 0 0"/>
-      <geometry>
-        <mesh filename="package://simple_robot_LIDAR/meshes/hokuyo.dae"/>
-      </geometry>
-    </visual>
-    <inertial>
-      <mass value="1e-5" />
-      <origin xyz="0 0 0" rpy="0 0 0"/>
-      <inertia ixx="1e-6" ixy="0" ixz="0" iyy="1e-6" iyz="0" izz="1e-6" />
-    </inertial>
+    <origin xyz="0.023 0 0.015" rpy="0 -1.571 -1.571" />
+    <parent link="camera_link" />
+    <child link="camera_point_link" />
+  </joint>
+  <link name="camera_point_link">
   </link>
   <joint name="hokuyo_joint" type="fixed">
@@ -203,4 +174,23 @@
 	 <dynamics damping="0.7"/>
   </joint>
+  <link name="hokuyo_link">
+    <collision>
+      <origin xyz="0 0 0" rpy="0 0 0"/>
+      <geometry>
+    <box size="0.1 0.1 0.1"/>
+      </geometry>
+    </collision>
+    <visual>
+      <origin xyz="0 0 0" rpy="0 0 0"/>
+      <geometry>
+        <mesh filename="package://simple_robot_LIDAR/meshes/hokuyo.dae"/>
+      </geometry>
+    </visual>
+    <inertial>
+      <mass value="1e-5" />
+      <origin xyz="0 0 0" rpy="0 0 0"/>
+      <inertia ixx="1e-6" ixy="0" ixz="0" iyy="1e-6" iyz="0" izz="1e-6" />
+    </inertial>
+  </link>
   <transmission name="left_wheel_transmission">
         <type>transmission_interface/SimpleTransmission</type>

Commit message: Add files via upload

File: urdf/robot_final.xacro (robot description, xacro)
@@ -26,5 +26,5 @@
   </link>
   <joint name="left_wheel_joint" type="continuous">
-    <origin xyz="0 -0.1005 0.09" rpy="1.5708 0 0" />
+    <origin xyz="0 0.1005 0.09" rpy="1.571 0 ${PI}" />
     <parent link="base_link" />
     <child link="left_wheel_link" />
@@ -52,5 +52,5 @@
   </link>
   <joint name="right_wheel_joint" type="continuous">
-    <origin xyz="0 0.1005 0.09" rpy="1.5708 0 0" />
+    <origin xyz="0 -0.1005 0.09" rpy="1.571 0 ${PI}" />
     <parent link="base_link" />
     <child link="right_wheel_link" />
